Commit message: update the project 2

File: Project2/catkin_ws/src/my_robot/urdf/my_robot.xacro (robot description, xacro)
@@ -72,5 +72,5 @@
       </geometry>
     </collision>
-    <visual name='visual'>
+    <visual name='front_left_wheel_visual'>
       <origin xyz="0 0 0" rpy="0 1.5707 1.5707" />
       <geometry>
@@ -94,5 +94,5 @@
       </geometry>
     </collision>
-    <visual name='visual'>
+    <visual name='front_right_wheel_visual'>
       <origin xyz="0 0 0" rpy="0 1.5707 1.5707" />
       <geometry>
@@ -117,5 +117,5 @@
       </geometry>
     </collision>
-    <visual name='visual'>
+    <visual name='rear_left_wheel_visual'>
       <origin xyz="0 0 0" rpy="0 1.5707 1.5707" />
       <geometry>
@@ -139,5 +139,5 @@
       </geometry>
     </collision>
-    <visual name='visual'>
+    <visual name='rear_right_wheel_visual'>
       <origin xyz="0 0 0" rpy="0 1.5707 1.5707" />
       <geometry>
@@ -232,3 +232,15 @@
     <axis xyz="0 1 0" rpy="0 0 0"/>
   </joint>
+  <gazebo reference="front_left_wheel">
+   <material>Gazebo/Red</material>
+  </gazebo>
+  <gazebo reference="front_right_wheel">
+   <material>Gazebo/Red</material>
+  </gazebo>
+  <gazebo reference="rear_left_wheel">
+   <material>Gazebo/Blue</material>
+  </gazebo>
+  <gazebo reference="rear_right_wheel">
+   <material>Gazebo/Blue</material>
+  </gazebo>
 </robot>
